File: Hardware/SGP30 Breakout.sch (EAGLE design)
At the start: 26 parts, among them J3 PTH, Q1 MOSFET-NCH-BSS138, Q2 MOSFET-NCH-BSS138, U1 SGP30, U2 MIC5504

Commit message: added section labels
Other:
- note added: "Bi-Directional Level Shifter"
- note added: "Connectors"
- note added: "SGP30"
- note added: "Voltage Regulator"
- moved on the sheet: C1, C2, C4, D1, J2, J3, J4, Q1, Q2, R1, R2, R3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

Commit message: fixed missing ground connection
Parts:
- U2: value MIC5504 -> AP2112k
Connections:
- removed net N$6: U2.GND
- net GND: now also U2.GND
Changed lines of the file:
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@@
 <part name="SUPPLY3" library="SparkFun-PowerSymbols" deviceset="3.3V" device=""/>
 <part name="SUPPLY5" library="SparkFun-PowerSymbols" deviceset="1.8V" device=""/>
-<part name="U2" library="SGP30" deviceset="MIC5504" device=""/>
+<part name="U2" library="SGP30" deviceset="MIC5504" device="" value="AP2112k"/>
 <part name="GND2" library="SparkFun" deviceset="GND" device=""/>
 <part name="Q1" library="SparkFun-DiscreteSemi" deviceset="MOSFET-NCH" device="-BSS138" value=""/>
@@
 </segment>
 <segment>
-<wire x1="50.8" y1="149.86" x2="50.8" y2="147.32" width="0.1524" layer="91"/>
-<pinref part="GND2" gate="1" pin="GND"/>
-</segment>
-<segment>
 <wire x1="40.64" y1="152.4" x2="40.64" y2="149.86" width="0.1524" layer="91"/>
 <pinref part="GND5" gate="1" pin="GND"/>
@@
 <pinref part="GND9" gate="1" pin="GND"/>
 <pinref part="C2" gate="G$1" pin="2"/>
+</segment>
+<segment>
+<pinref part="GND2" gate="1" pin="GND"/>
+<wire x1="50.8" y1="147.32" x2="50.8" y2="149.86" width="0.1524" layer="91"/>
+<pinref part="U2" gate="G$1" pin="GND"/>
+<wire x1="50.8" y1="149.86" x2="53.34" y2="149.86" width="0.1524" layer="91"/>
 </segment>
 </net>
@@
 </segment>
 </net>
-<net name="N$6" class="0">
-<segment>
-<pinref part="U2" gate="G$1" pin="GND"/>
-<wire x1="53.34" y1="149.86" x2="50.8" y2="149.86" width="0.1524" layer="91"/>
-</segment>
-</net>

Commit message: Fixed ground connections
* Pad not grounded
* Connected pad to solde mask
Parts:
- added U$9: QWIIC_LOGO_7MM, SparkFun-Aesthetics:QWIIC_LOGO_7MM
